File: untitled2.kicad_sch (KiCad schematic)
At the start: 6 parts, among them P3 USB_C_Plug_USB2.0, U3 NCP1117-3.3_SOT223

Commit message: Add files via upload
PCB design as of april first
Parts:
- removed U3: NCP1117-3.3_SOT223, Package_TO_SOT_SMD:SOT-223-3_TabPin2, symbol Regulator_Linear:NCP1117-3.3_SOT223
- added U5: NCP1117-3.3_SOT223, Package_TO_SOT_SMD:SOT-223-3_TabPin2, symbol Regulator_Linear:NCP1117-3.3_SOT223
- renumbered C2 to C34, C6 to C35, P3 to P4, R3 to R15, R4 to R16
Connections:
- net +3V3: now also U5.2 (VO)
- net GND: now also U5.1 (GND)
- net VBUS: now also U5.3 (VI)
- net USB_D+ renamed USB_D+2
- net USB_D- renamed USB_D-2
