File: IEEE Keyboard Project.kicad_pcb (KiCad board)
At the start: 2 copper layers, 353.5 x 145.7 mm, 203 parts, among them J1 Conn_01x04_Socket, J2 Conn_01x04_Socket, P3 USB_C_Plug_USB2.0, P4 USB_C_Plug_USB2.0, SW1 SW_Push, SW2 SW_Push, SW3 SW_Push, SW4 SW_Push, SW5 SW_Nidec_CAS-120A1, U1 RP2354B, U2 RP2354B, U3 NCP1117-3.3_SOT223, U4 NCP1117-3.3_SOT223, U5 NCP1117-3.3_SOT223, Y1 ABM8-272-T3, Y2 ABM8-272-T3, Y5 ABM8-272-T3, Y6 ABM8-272-T3

Commit message: Add files via upload
Parts:
- removed S13, S14, S15, S16, S17, S18, S19, S20, S21, S22, S23, S24, S25, S26, S27, S28, S4: , ceoloide:switch_mx
- D31, D32, D33, D34, D35, D36, D37, D38, D39, D40, D41, D42, D43, D44, D45, D46, D47, D48, D49, D50, D51, D52, D53, D54, D55, D56: moved to B.Cu
- moved MX39 267.2 mm to (325.0, 91.0), turned to 20 degrees
- moved MX40 262.5 mm to (331.5, 109.1), turned to 20 degrees
- moved MX42 259.1 mm to (298.5, 74.5), turned to 20 degrees
- moved MX41 257.5 mm to (291.9, 56.1), turned to 20 degrees
- moved MX45 206.1 mm to (275.5, 68.0), turned to 20 degrees
- moved MX49 202.7 mm to (302.4, 142.6), turned to 20 degrees
- moved MX48 200.1 mm to (295.4, 123.5), turned to 20 degrees
- moved MX47 197.6 mm to (288.9, 105.1), turned to 20 degrees
- moved MX52 195.3 mm to (271.9, 114.6), turned to 20 degrees
- moved MX44 191.6 mm to (311.5, 111.0), turned to 20 degrees
- moved MX46 181.9 mm to (282.1, 86.4), turned to 20 degrees
- moved D30 176.4 mm to (357.2, 75.5)
- moved D32 174.7 mm to (370.7, 112.0), turned to 180 degrees
- moved D33 164.2 mm to (332.8, 63.5), turned to 180 degrees
- moved MX43 162.6 mm to (305.1, 92.6), turned to 20 degrees
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Other:
- board size 353.5 x 145.7 mm -> 353.8 x 147.9 mm
