File: IEEE Keyboard Project.kicad_pcb (KiCad board)
At the start: 2 copper layers, 353.5 x 145.7 mm, 58 parts

Commit message: Add files via upload
PCB design as of april first
Parts:
- removed LOGO1 (x2): , ceoloide:utility_ergogen_logo
- removed the S1 at (53.4, 101.6)
- removed the S10 at (98.0, 90.2)
- removed the S11 at (104.5, 72.3)
- removed the S12 at (111.0, 54.5)
- removed the S13 at (111.1, 109.9)
- removed the S14 at (117.6, 92.0)
- removed the S15 at (124.1, 74.1)
- removed the S16 at (130.6, 56.3)
- removed the S17 at (126.9, 122.0)
- removed the S18 at (133.4, 104.1)
- removed the S19 at (139.9, 86.3)
- removed the S2 at (59.9, 83.8)
- removed the S20 at (146.4, 68.4)
- removed the S21 at (143.4, 132.2)
- removed the S22 at (149.9, 114.4)
- removed the S23 at (156.4, 96.5)
- removed the S24 at (162.9, 78.7)
- removed the S25 at (113.2, 141.8)
- removed the S26 at (131.6, 148.5)
- removed the S27 at (156.4, 161.9)
- removed the S28 at (167.4, 146.4)
- removed the S3 at (66.4, 65.9)
- removed the S5 at (71.3, 108.1)
- removed the S6 at (77.8, 90.3)
- removed the S7 at (84.3, 72.4)
- removed the S8 at (90.8, 54.6)
- removed the S9 at (91.5, 108.1)
- added C10: 4.7u, Capacitor_SMD:C_0402_1005Metric, F.Cu at (215.0, 205.4)
- added C11: 100n, Capacitor_SMD:C_0402_1005Metric, F.Cu at (215.0, 207.3)
- added C12: 100n, Capacitor_SMD:C_0402_1005Metric, F.Cu at (215.0, 209.3)
- added C13: 100n, Capacitor_SMD:C_0402_1005Metric, F.Cu at (217.9, 197.4)
- added C14: 100n, Capacitor_SMD:C_0402_1005Metric, F.Cu at (217.9, 199.5)
- added C15: 100n, Capacitor_SMD:C_0402_1005Metric, F.Cu at (217.9, 201.4)
- added C16: 100n, Capacitor_SMD:C_0402_1005Metric, F.Cu at (217.9, 203.4)
- added C17: 100n, Capacitor_SMD:C_0402_1005Metric, F.Cu at (217.9, 205.4)
- added C18: 100n, Capacitor_SMD:C_0402_1005Metric, F.Cu at (217.9, 207.3)
- added C2: 10u, Capacitor_SMD:C_0805_2012Metric, F.Cu at (239.8, 198.0)
- added C20: 15p, Capacitor_SMD:C_0402_1005Metric, F.Cu at (217.9, 209.3)
- added C20: 15p, Capacitor_SMD:C_0402_1005Metric, F.Cu at (216.9, 244.5)
- added C22: 100n, Capacitor_SMD:C_0402_1005Metric, F.Cu at (220.8, 197.5)
- added C23: 100n, Capacitor_SMD:C_0402_1005Metric, F.Cu at (220.8, 199.5)
- added C24: 100n, Capacitor_SMD:C_0402_1005Metric, F.Cu at (220.8, 201.4)
- added C25: 100n, Capacitor_SMD:C_0402_1005Metric, F.Cu at (220.8, 203.4)
- added C26: 4.7u, Capacitor_SMD:C_0402_1005Metric, F.Cu at (220.8, 205.4)
- added C27: 4.7u, Capacitor_SMD:C_0402_1005Metric, F.Cu at (220.8, 207.3)
- added C28: 100n, Capacitor_SMD:C_0402_1005Metric, F.Cu at (220.8, 209.3)
- added C29: 4.7u, Capacitor_SMD:C_0402_1005Metric, F.Cu at (223.6, 197.5)
- added C3: 15p, Capacitor_SMD:C_0402_1005Metric, F.Cu at (229.1, 189.7)
- added C30: 100n, Capacitor_SMD:C_0402_1005Metric, F.Cu at (223.6, 199.5)
- added C31: 100n, Capacitor_SMD:C_0402_1005Metric, F.Cu at (223.6, 201.4)
- added C32: 100n, Capacitor_SMD:C_0402_1005Metric, F.Cu at (223.6, 203.4)
- added C33: 100n, Capacitor_SMD:C_0402_1005Metric, F.Cu at (223.6, 205.4)
- added C34: 10u, Capacitor_SMD:C_0805_2012Metric, F.Cu at (239.8, 208.3)
- added C35: 10u, Capacitor_SMD:C_0805_2012Metric, F.Cu at (239.8, 211.3)
- added C36: 4.7u, Capacitor_SMD:C_0402_1005Metric, F.Cu at (256.2, 189.2)
- added C37: 4.7u, Capacitor_SMD:C_0402_1005Metric, F.Cu at (256.2, 191.2)
- added C38: 4.7u, Capacitor_SMD:C_0402_1005Metric, F.Cu at (256.2, 193.2)
- added C39: 4.7u, Capacitor_SMD:C_0402_1005Metric, F.Cu at (256.2, 195.1)
- added C4: 15p, Capacitor_SMD:C_0402_1005Metric, F.Cu at (215.0, 199.5)
- added C5: 15p, Capacitor_SMD:C_0402_1005Metric, F.Cu at (216.9, 242.5)
- added C5: 15p, Capacitor_SMD:C_0402_1005Metric, F.Cu at (215.0, 201.4)
- added C6: 10u, Capacitor_SMD:C_0805_2012Metric, F.Cu at (239.8, 201.0)
- added C8: 100n, Capacitor_SMD:C_0402_1005Metric, F.Cu at (215.0, 203.4)
- added D1: D_Small, Diode_SMD:D_01005_0402Metric, B.Cu at (64.5, 43.0)
- added D10: D_Small, Diode_SMD:D_01005_0402Metric, F.Cu at (212.3, 182.3)
- added D11: D_Small, Diode_SMD:D_01005_0402Metric, F.Cu at (76.8, 64.0)
- added D12: D_Small, Diode_SMD:D_01005_0402Metric, F.Cu at (214.8, 169.2)
- added D13: D_Small, Diode_SMD:D_01005_0402Metric, F.Cu at (214.8, 170.8)
- added D14: D_Small, Diode_SMD:D_01005_0402Metric, F.Cu at (214.8, 172.4)
- added D15: D_Small, Diode_SMD:D_01005_0402Metric, F.Cu at (214.8, 174.1)
- added D16: D_Small, Diode_SMD:D_01005_0402Metric, F.Cu at (214.8, 175.8)
- added D17: D_Small, Diode_SMD:D_01005_0402Metric, F.Cu at (214.8, 177.4)
- added D18: D_Small, Diode_SMD:D_01005_0402Metric, F.Cu at (214.8, 179.1)
- added D19: D_Small, Diode_SMD:D_01005_0402Metric, F.Cu at (214.8, 180.7)
- added D2: D_Small, Diode_SMD:D_01005_0402Metric, F.Cu at (212.3, 169.2)
- added D20: D_Small, Diode_SMD:D_01005_0402Metric, F.Cu at (214.8, 182.3)
- added D21: D_Small, Diode_SMD:D_01005_0402Metric, F.Cu at (217.2, 167.5)
- added D22: D_Small, Diode_SMD:D_01005_0402Metric, F.Cu at (217.2, 169.2)
- added D23: D_Small, Diode_SMD:D_01005_0402Metric, F.Cu at (217.2, 170.8)
- added D24: D_Small, Diode_SMD:D_01005_0402Metric, F.Cu at (217.2, 172.4)
- added D25: D_Small, Diode_SMD:D_01005_0402Metric, F.Cu at (217.2, 174.1)
- added D26: D_Small, Diode_SMD:D_01005_0402Metric, F.Cu at (217.2, 175.8)
- added D27: D_Small, Diode_SMD:D_01005_0402Metric, F.Cu at (217.2, 177.4)
- added D28: D_Small, Diode_SMD:D_01005_0402Metric, F.Cu at (217.2, 179.1)
- added D29: D_Small, Diode_SMD:D_01005_0402Metric, F.Cu at (217.2, 180.7)
- added D3: D_Small, Diode_SMD:D_01005_0402Metric, F.Cu at (212.3, 170.8)
- added D30: D_Small, Diode_SMD:D_01005_0402Metric, F.Cu at (217.2, 182.3)
- added D31: D_Small, Diode_SMD:D_01005_0402Metric, F.Cu at (219.7, 167.5)
- added D32: D_Small, Diode_SMD:D_01005_0402Metric, F.Cu at (219.7, 169.2)
- added D33: D_Small, Diode_SMD:D_01005_0402Metric, F.Cu at (219.7, 170.8)
- added D34: D_Small, Diode_SMD:D_01005_0402Metric, F.Cu at (219.7, 172.4)
- added D35: D_Small, Diode_SMD:D_01005_0402Metric, F.Cu at (219.7, 174.1)
- added D36: D_Small, Diode_SMD:D_01005_0402Metric, F.Cu at (219.7, 175.8)
- added D37: D_Small, Diode_SMD:D_01005_0402Metric, F.Cu at (219.7, 177.4)
- added D38: D_Small, Diode_SMD:D_01005_0402Metric, F.Cu at (219.7, 179.1)
- added D39: D_Small, Diode_SMD:D_01005_0402Metric, F.Cu at (219.7, 180.7)
- added D4: D_Small, Diode_SMD:D_01005_0402Metric, F.Cu at (212.3, 172.4)
- added D40: D_Small, Diode_SMD:D_01005_0402Metric, F.Cu at (219.7, 182.3)
- added D41: D_Small, Diode_SMD:D_01005_0402Metric, F.Cu at (222.2, 167.5)
- added D42: D_Small, Diode_SMD:D_01005_0402Metric, F.Cu at (222.2, 169.2)
- added D43: D_Small, Diode_SMD:D_01005_0402Metric, F.Cu at (222.2, 170.8)
- added D44: D_Small, Diode_SMD:D_01005_0402Metric, F.Cu at (222.2, 172.4)
- added D45: D_Small, Diode_SMD:D_01005_0402Metric, F.Cu at (222.2, 174.1)
- added D46: D_Small, Diode_SMD:D_01005_0402Metric, F.Cu at (222.2, 175.8)
- added D47: D_Small, Diode_SMD:D_01005_0402Metric, F.Cu at (222.2, 177.4)
- added D48: D_Small, Diode_SMD:D_01005_0402Metric, F.Cu at (222.2, 179.1)
- added D49: D_Small, Diode_SMD:D_01005_0402Metric, F.Cu at (222.2, 180.7)
- added D5: D_Small, Diode_SMD:D_01005_0402Metric, F.Cu at (212.3, 174.1)
- added D50: D_Small, Diode_SMD:D_01005_0402Metric, F.Cu at (222.2, 182.3)
- added D51: D_Small, Diode_SMD:D_01005_0402Metric, F.Cu at (224.7, 167.5)
- added D52: D_Small, Diode_SMD:D_01005_0402Metric, F.Cu at (224.7, 169.2)
- added D53: D_Small, Diode_SMD:D_01005_0402Metric, F.Cu at (224.7, 170.8)
- added D54: D_Small, Diode_SMD:D_01005_0402Metric, F.Cu at (224.7, 172.4)
- added D55: D_Small, Diode_SMD:D_01005_0402Metric, F.Cu at (224.7, 174.1)
- added D56: D_Small, Diode_SMD:D_01005_0402Metric, F.Cu at (224.7, 175.8)
- added D6: D_Small, Diode_SMD:D_01005_0402Metric, F.Cu at (212.3, 175.8)
- added D7: D_Small, Diode_SMD:D_01005_0402Metric, F.Cu at (212.3, 177.4)
- added D8: D_Small, Diode_SMD:D_01005_0402Metric, F.Cu at (212.3, 179.1)
- added D9: D_Small, Diode_SMD:D_01005_0402Metric, F.Cu at (212.3, 180.7)
- added J1: Conn_01x04_Socket, Connector_JST:JST_EH_S4B-EH_1x04_P2.50mm_Horizontal, F.Cu at (244.5, 224.9)
- added J2: Conn_01x04_Socket, Connector_JST:JST_EH_S4B-EH_1x04_P2.50mm_Horizontal, F.Cu at (240.7, 237.9)
- added L3: 3.3u, Inductor_SMD:L_Coilcraft_LPS3314, F.Cu at (252.2, 190.9)
- added L4: 3.3u, Inductor_SMD:L_Coilcraft_LPS3314, F.Cu at (252.2, 196.1)
- added MX1: MX_SW_HS, Button_Switch_Keyboard:SW_Cherry_MX_1.00u_PCB, F.Cu at (75.5, 43.3)
- added MX10: MX_SW_HS, Button_Switch_Keyboard:SW_Cherry_MX_1.00u_PCB, F.Cu at (127.6, 69.6)
- added MX11: MX_SW_HS, Button_Switch_Keyboard:SW_Cherry_MX_1.00u_PCB, F.Cu at (144.1, 82.1)
- added MX12: MX_SW_HS, Button_Switch_Keyboard:SW_Cherry_MX_1.00u_PCB, F.Cu at (161.3, 92.3)
- added MX13: MX_SW_HS, Button_Switch_Keyboard:SW_Cherry_MX_1.00u_PCB, F.Cu at (62.3, 79.6)
- added MX14: MX_SW_HS, Button_Switch_Keyboard:SW_Cherry_MX_1.00u_PCB, F.Cu at (80.5, 86.3)
- added MX15: MX_SW_HS, Button_Switch_Keyboard:SW_Cherry_MX_1.00u_PCB, F.Cu at (101.3, 85.9)
- added MX16: MX_SW_HS, Button_Switch_Keyboard:SW_Cherry_MX_1.00u_PCB, F.Cu at (121.3, 87.8)
- added MX17: MX_SW_HS, Button_Switch_Keyboard:SW_Cherry_MX_1.00u_PCB, F.Cu at (137.5, 100.5)
- added MX18: MX_SW_HS, Button_Switch_Keyboard:SW_Cherry_MX_1.00u_PCB, F.Cu at (154.4, 110.4)
- added MX19: MX_SW_HS, Button_Switch_Keyboard:SW_Cherry_MX_1.00u_PCB, F.Cu at (55.5, 97.9)
- added MX2: MX_SW_HS, Button_Switch_Keyboard:SW_Cherry_MX_1.00u_PCB, F.Cu at (93.9, 49.9)
- added MX20: MX_SW_HS, Button_Switch_Keyboard:SW_Cherry_MX_1.00u_PCB, F.Cu at (73.9, 104.4)
- added MX21: MX_SW_HS, Button_Switch_Keyboard:SW_Cherry_MX_1.00u_PCB, F.Cu at (94.5, 104.0)
- added MX22: MX_SW_HS, Button_Switch_Keyboard:SW_Cherry_MX_1.00u_PCB, F.Cu at (114.8, 106.0)
- added MX23: MX_SW_HS, Button_Switch_Keyboard:SW_Cherry_MX_1.00u_PCB, F.Cu at (130.6, 119.1)
- added MX24: MX_SW_HS, Button_Switch_Keyboard:SW_Cherry_MX_1.00u_PCB, F.Cu at (147.9, 128.9)
- added MX25: MX_SW_HS, Button_Switch_Keyboard:SW_Cherry_MX_1.00u_PCB, F.Cu at (123.9, 137.4)
- added MX26: MX_SW_HS, Button_Switch_Keyboard:SW_Cherry_MX_1.00u_PCB, F.Cu at (141.2, 147.3)
- added MX27: MX_SW_HS, Button_Switch_Keyboard:SW_Cherry_MX_1.00u_PCB, F.Cu at (172.7, 143.0)
- added MX28: MX_SW_HS, Button_Switch_Keyboard:SW_Cherry_MX_1.00u_PCB, F.Cu at (161.5, 158.8)
- added MX29: MX_SW_HS, Button_Switch_Keyboard:SW_Cherry_MX_1.00u_PCB, F.Cu at (139.7, 183.0)
- added MX3: MX_SW_HS, Button_Switch_Keyboard:SW_Cherry_MX_1.00u_PCB, F.Cu at (114.4, 49.6)
- added MX30: MX_SW_HS, Button_Switch_Keyboard:SW_Cherry_MX_1.00u_PCB, F.Cu at (139.7, 198.1)
- added MX31: MX_SW_HS, Button_Switch_Keyboard:SW_Cherry_MX_1.00u_PCB, F.Cu at (117.4, 213.1)
- added MX32: MX_SW_HS, Button_Switch_Keyboard:SW_Cherry_MX_1.00u_PCB, F.Cu at (101.1, 232.9)
- added MX33: MX_SW_HS, Button_Switch_Keyboard:SW_Cherry_MX_1.00u_PCB, F.Cu at (24.5, 206.9)
- added MX34: MX_SW_HS, Button_Switch_Keyboard:SW_Cherry_MX_1.00u_PCB, F.Cu at (60.6, 184.4)
- added MX35: MX_SW_HS, Button_Switch_Keyboard:SW_Cherry_MX_1.00u_PCB, F.Cu at (5.54, 162.4)
- added MX36: MX_SW_HS, Button_Switch_Keyboard:SW_Cherry_MX_1.00u_PCB, F.Cu at (-50.5, 155.1)
- added MX37: MX_SW_HS, Button_Switch_Keyboard:SW_Cherry_MX_1.00u_PCB, F.Cu at (154.8, 198.1)
- added MX38: MX_SW_HS, Button_Switch_Keyboard:SW_Cherry_MX_1.00u_PCB, F.Cu at (132.5, 213.1)
- added MX39: MX_SW_HS, Button_Switch_Keyboard:SW_Cherry_MX_1.00u_PCB, F.Cu at (132.5, 228.2)
- added MX4: MX_SW_HS, Button_Switch_Keyboard:SW_Cherry_MX_1.00u_PCB, F.Cu at (134.5, 51.5)
- added MX40: MX_SW_HS, Button_Switch_Keyboard:SW_Cherry_MX_1.00u_PCB, F.Cu at (132.5, 243.3)
- added MX41: MX_SW_HS, Button_Switch_Keyboard:SW_Cherry_MX_1.00u_PCB, F.Cu at (132.5, 258.4)
- added MX42: MX_SW_HS, Button_Switch_Keyboard:SW_Cherry_MX_1.00u_PCB, F.Cu at (132.5, 273.5)
- added MX43: MX_SW_HS, Button_Switch_Keyboard:SW_Cherry_MX_1.00u_PCB, F.Cu at (169.9, 183.0)
- added MX44: MX_SW_HS, Button_Switch_Keyboard:SW_Cherry_MX_1.00u_PCB, F.Cu at (169.9, 198.1)
- added MX45: MX_SW_HS, Button_Switch_Keyboard:SW_Cherry_MX_1.00u_PCB, F.Cu at (147.6, 213.1)
- added MX46: MX_SW_HS, Button_Switch_Keyboard:SW_Cherry_MX_1.00u_PCB, F.Cu at (147.6, 228.2)
- added MX47: MX_SW_HS, Button_Switch_Keyboard:SW_Cherry_MX_1.00u_PCB, F.Cu at (147.6, 243.3)
- added MX48: MX_SW_HS, Button_Switch_Keyboard:SW_Cherry_MX_1.00u_PCB, F.Cu at (147.6, 258.4)
- added MX49: MX_SW_HS, Button_Switch_Keyboard:SW_Cherry_MX_1.00u_PCB, F.Cu at (147.6, 273.5)
- added MX5: MX_SW_HS, Button_Switch_Keyboard:SW_Cherry_MX_1.00u_PCB, F.Cu at (151.0, 64.0)
- added MX50: MX_SW_HS, Button_Switch_Keyboard:SW_Cherry_MX_1.00u_PCB, F.Cu at (185.0, 183.0)
- added MX51: MX_SW_HS, Button_Switch_Keyboard:SW_Cherry_MX_1.00u_PCB, F.Cu at (185.0, 198.1)
- added MX52: MX_SW_HS, Button_Switch_Keyboard:SW_Cherry_MX_1.00u_PCB, F.Cu at (162.7, 213.1)
- added MX53: MX_SW_HS, Button_Switch_Keyboard:SW_Cherry_MX_1.00u_PCB, F.Cu at (162.7, 228.2)
- added MX54: MX_SW_HS, Button_Switch_Keyboard:SW_Cherry_MX_1.00u_PCB, F.Cu at (162.7, 243.3)
- added MX55: MX_SW_HS, Button_Switch_Keyboard:SW_Cherry_MX_1.00u_PCB, F.Cu at (162.7, 258.4)
- added MX56: MX_SW_HS, Button_Switch_Keyboard:SW_Cherry_MX_1.00u_PCB, F.Cu at (162.7, 273.5)
- added MX6: MX_SW_HS, Button_Switch_Keyboard:SW_Cherry_MX_1.00u_PCB, F.Cu at (168.1, 74.1)
- added MX7: MX_SW_HS, Button_Switch_Keyboard:SW_Cherry_MX_1.00u_PCB, F.Cu at (68.9, 61.5)
- added MX8: MX_SW_HS, Button_Switch_Keyboard:SW_Cherry_MX_1.00u_PCB, F.Cu at (87.0, 68.0)
- added MX9: MX_SW_HS, Button_Switch_Keyboard:SW_Cherry_MX_1.00u_PCB, F.Cu at (107.8, 67.6)
- added P3: USB_C_Plug_USB2.0, 2340901-1:TE_2340901-1, F.Cu at (284.4, 254.8)
- added P4: USB_C_Plug_USB2.0, 2340901-1:TE_2340901-1, F.Cu at (289.1, 266.5)
- added R1: 27, Resistor_SMD:R_0402_1005Metric, F.Cu at (202.4, 222.0)
- added R10: 1k, Resistor_SMD:R_0402_1005Metric, F.Cu at (205.3, 228.0)
- added R11: 33, Resistor_SMD:R_0402_1005Metric, F.Cu at (208.2, 222.0)
- added R12: 1k, Resistor_SMD:R_0402_1005Metric, F.Cu at (208.2, 224.0)
- added R12: 1k, Resistor_SMD:R_0402_1005Metric, F.Cu at (219.8, 242.5)
- added R13: 27, Resistor_SMD:R_0402_1005Metric, F.Cu at (208.2, 226.0)
- added R14: 27, Resistor_SMD:R_0402_1005Metric, F.Cu at (208.2, 228.0)
- added R15: 1k, Resistor_SMD:R_0402_1005Metric, F.Cu at (278.9, 274.7)
- added R16: 1k, Resistor_SMD:R_0402_1005Metric, F.Cu at (278.9, 276.7)
- added R2: 27, Resistor_SMD:R_0402_1005Metric, F.Cu at (202.4, 224.0)
- added R3: 1k, Resistor_SMD:R_0402_1005Metric, F.Cu at (278.9, 258.7)
- added R4: 1k, Resistor_SMD:R_0402_1005Metric, F.Cu at (278.9, 260.7)
- added R5: 33, Resistor_SMD:R_0402_1005Metric, F.Cu at (202.4, 226.0)
- added R6: 1k, Resistor_SMD:R_0402_1005Metric, F.Cu at (202.4, 228.0)
- added R7: 1k, Resistor_SMD:R_0402_1005Metric, F.Cu at (205.3, 222.0)
- added R8: 1k, Resistor_SMD:R_0402_1005Metric, F.Cu at (205.3, 224.0)
- added R9: 1k, Resistor_SMD:R_0402_1005Metric, F.Cu at (205.3, 226.0)
- added SW1: SW_Push, Button_Switch_SMD:SW_Push_1P1T_NO_Vertical_Wuerth_434133025816, F.Cu at (216.9, 212.7)
- added SW2: SW_Push, Button_Switch_SMD:SW_Push_1P1T_NO_Vertical_Wuerth_434133025816, F.Cu at (216.9, 217.4)
- added SW3: SW_Push, Button_Switch_SMD:SW_Push_1P1T_NO_Vertical_Wuerth_434133025816, F.Cu at (216.9, 222.2)
- added SW4: SW_Push, Button_Switch_SMD:SW_Push_1P1T_NO_Vertical_Wuerth_434133025816, F.Cu at (216.9, 226.9)
- added SW5: SW_Nidec_CAS-120A1, Button_Switch_SMD:Nidec_Copal_CAS-120A, F.Cu at (223.1, 222.9)
- added U1: RP2354B, Package_DFN_QFN:QFN-80-1EP_10x10mm_P0.4mm_EP3.4x3.4mm, F.Cu at (172.0, 123.5)
- added U2: RP2354B, Package_DFN_QFN:QFN-80-1EP_10x10mm_P0.4mm_EP3.4x3.4mm, F.Cu at (207.5, 214.9)
- added U3: NCP1117-3.3_SOT223, Package_TO_SOT_SMD:SOT-223-3_TabPin2, F.Cu at (232.7, 200.7)
- added U3: NCP1117-3.3_SOT223, Package_TO_SOT_SMD:SOT-223-3_TabPin2, F.Cu at (262.5, 221.4)
- added U4: NCP1117-3.3_SOT223, Package_TO_SOT_SMD:SOT-223-3_TabPin2, F.Cu at (232.7, 211.0)
- added U5: NCP1117-3.3_SOT223, Package_TO_SOT_SMD:SOT-223-3_TabPin2, F.Cu at (262.5, 231.7)
- added Y1: ABM8-272-T3, Crystal:Crystal_SMD_3225-4Pin_3.2x2.5mm, F.Cu at (222.9, 212.6)
- added Y2: ABM8-272-T3, Crystal:Crystal_SMD_3225-4Pin_3.2x2.5mm, F.Cu at (222.9, 217.1)
- added Y5: ABM8-272-T3, ABM8-272-T3:XTAL_ABM8-272-T3, F.Cu at (218.3, 239.0)
- added Y6: ABM8-272-T3, ABM8-272-T3:XTAL_ABM8-272-T3, F.Cu at (223.3, 239.0)
- S4: moved to F.Cu
- moved S4 138.2 mm to (97.6, -87.9), turned to 180 degrees
Other:
- outline, holes or cut-outs redrawn
- board text removed: "JLCJLCJLCJLC"

Commit message: Add files via upload
Parts:
- removed S24: , ceoloide:switch_mx
- removed U3 (x2): NCP1117-3.3_SOT223, Package_TO_SOT_SMD:SOT-223-3_TabPin2
- added D10: D_Small, Diode_SMD:D_01005_0402Metric, B.Cu at (122.3, 77.0)
- added D12: D_Small, Diode_SMD:D_01005_0402Metric, B.Cu at (156.2, 100.0)
- added D13: D_Small, Diode_SMD:D_01005_0402Metric, B.Cu at (56.8, 87.0)
- added D14: D_Small, Diode_SMD:D_01005_0402Metric, B.Cu at (75.2, 94.0)
- added D15: D_Small, Diode_SMD:D_01005_0402Metric, B.Cu at (96.3, 93.5)
- added D16: D_Small, Diode_SMD:D_01005_0402Metric, B.Cu at (116.0, 95.5)
- added D17: D_Small, Diode_SMD:D_01005_0402Metric, B.Cu at (132.5, 108.0)
- added D18: D_Small, Diode_SMD:D_01005_0402Metric, B.Cu at (149.2, 118.0)
- added D19: D_Small, Diode_SMD:D_01005_0402Metric, B.Cu at (50.3, 105.5)
- added D2: D_Small, Diode_SMD:D_01005_0402Metric, B.Cu at (88.2, 57.5)
- added D20: D_Small, Diode_SMD:D_01005_0402Metric, B.Cu at (68.8, 112.0)
- added D21: D_Small, Diode_SMD:D_01005_0402Metric, B.Cu at (89.0, 111.5)
- added D22: D_Small, Diode_SMD:D_01005_0402Metric, B.Cu at (109.8, 113.5)
- added D23: D_Small, Diode_SMD:D_01005_0402Metric, B.Cu at (125.3, 126.5)
- added D24: D_Small, Diode_SMD:D_01005_0402Metric, B.Cu at (142.8, 136.5)
- added D25: D_Small, Diode_SMD:D_01005_0402Metric, B.Cu at (118.3, 145.0)
- added D26: D_Small, Diode_SMD:D_01005_0402Metric, B.Cu at (136.3, 155.0)
- added D27: D_Small, Diode_SMD:D_01005_0402Metric, B.Cu at (165.8, 148.5)
- added D28: D_Small, Diode_SMD:D_01005_0402Metric, B.Cu at (154.3, 164.5)
- added D3: D_Small, Diode_SMD:D_01005_0402Metric, B.Cu at (109.7, 57.5)
- added D4: D_Small, Diode_SMD:D_01005_0402Metric, B.Cu at (129.2, 59.0)
- added D5: D_Small, Diode_SMD:D_01005_0402Metric, B.Cu at (145.8, 71.5)
- added D6: D_Small, Diode_SMD:D_01005_0402Metric, B.Cu at (163.0, 81.5)
- added D7: D_Small, Diode_SMD:D_01005_0402Metric, B.Cu at (64.3, 69.0)
- added D8: D_Small, Diode_SMD:D_01005_0402Metric, B.Cu at (81.5, 75.5)
- added D9: D_Small, Diode_SMD:D_01005_0402Metric, B.Cu at (102.8, 75.0)
- moved P3 190.7 mm to (179.5, 95.5), turned to 160 degrees
- moved P4 171.8 mm to (245.5, 100.3), turned to -160 degrees
- moved U1 149.8 mm to (297.6, 205.1)
- moved J1 131.3 mm to (191.8, 104.6), turned to -110 degrees
- moved R14 125.1 mm to (331.5, 206.5)
- moved J2 123.4 mm to (238.0, 114.5), turned to 110 degrees
- moved R13 122.0 mm to (327.5, 200.5)
- moved SW4 117.1 mm to (167.4, 120.8), turned to -20 degrees
- moved SW3 107.6 mm to (174.4, 123.3), turned to -20 degrees
- moved SW5 105.8 mm to (180.5, 126.0), turned to -20 degrees
- moved SW2 81.7 mm to (298.6, 220.4), turned to 180 degrees
- moved R16 77.1 mm to (327.2, 216.7), turned to 90 degrees
- moved R15 74.3 mm to (325.2, 216.7), turned to 90 degrees
- moved L4 70.5 mm to (208.5, 251.5)
- moved Y5 69.5 mm to (286.1, 223.7)
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
Commit message: Sorting out components on PCB
Parts:
- removed the D10 at (209.3, 176.4)
- removed the D12 at (211.8, 163.2)
- removed the D13 at (211.8, 164.8)
- removed the D14 at (211.8, 166.5)
- removed the D15 at (211.8, 168.2)
- removed the D16 at (211.8, 169.8)
- removed the D17 at (211.8, 171.4)
- removed the D18 at (211.8, 173.1)
- removed the D19 at (211.8, 174.8)
- removed the D2 at (200.0, 163.0)
- removed the D20 at (211.8, 176.4)
- removed the D21 at (214.3, 161.6)
- removed the D22 at (214.3, 163.2)
- removed the D23 at (214.3, 164.8)
- removed the D24 at (214.3, 166.5)
- removed the D25 at (214.3, 168.2)
- removed the D26 at (214.3, 169.8)
- removed the D27 at (214.3, 171.4)
- removed the D28 at (214.3, 173.1)
- removed the D3 at (209.3, 164.8)
- removed the D4 at (209.3, 166.5)
- removed the D5 at (209.3, 168.2)
- removed the D6 at (209.3, 169.8)
- removed the D7 at (209.3, 171.4)
- removed the D8 at (209.3, 173.1)
- removed the D9 at (209.3, 174.8)
- removed S1, S10, S11, S12, S13, S14, S15, S16, S17, S18, S19, S2, S20, S21, S22, S23, S25, S26, S27, S28, S3, S4 (x2), S5, S6, S7, S8, S9: , ceoloide:switch_mx
- removed Y1: ABM8-272-T3, Crystal:Crystal_SMD_3225-4Pin_3.2x2.5mm
- D29, D30, D31, D32, D33, D34, D35, D36, D37, D38, D39, D40, D41, D42, D43, D44, D45, D46, D47, D48, D49, D50, D51, D52, D53, D54, D55, D56: moved to B.Cu
- moved MX36 424.7 mm to (371.8, 109.6), turned to 20 degrees
- moved MX35 366.5 mm to (365.0, 91.0), turned to 20 degrees
- moved MX33 361.3 mm to (351.8, 54.1), turned to 20 degrees
- moved MX34 318.0 mm to (358.3, 72.6), turned to 20 degrees
- moved MX32 317.0 mm to (390.1, 102.6), turned to 20 degrees
- moved MX31 295.6 mm to (383.3, 84.1), turned to 20 degrees
- moved MX42 272.0 mm to (318.0, 74.5), turned to 20 degrees
- moved MX30 271.3 mm to (376.6, 65.9), turned to 20 degrees
- moved MX41 270.0 mm to (311.3, 56.1), turned to 20 degrees
- moved MX29 267.2 mm to (370.0, 47.5), turned to 20 degrees
- moved MX40 256.4 mm to (351.0, 109.1), turned to 20 degrees
- moved MX39 252.5 mm to (344.5, 91.0), turned to 20 degrees
- moved MX38 248.8 mm to (337.8, 72.6), turned to 20 degrees
- moved MX37 227.7 mm to (331.1, 54.0), turned to 20 degrees
- moved MX49 217.9 mm to (321.8, 142.6), turned to 20 degrees
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Other:
- board size 353.5 x 145.7 mm -> 373.2 x 147.9 mm
- copper layers 2 -> 4
